File: octaver/octaver.kicad_sch (KiCad schematic)
At the start: 14 parts, among them Q1 2N3904, Q2 2N3904

Commit message: she is working?
Parts:
- removed C1, C2: 1, symbol Device:C
- removed L1: 1k, symbol Device:L
- removed Q1, Q2: 2N3904, Package_TO_SOT_THT:TO-92_Inline, symbol Transistor_BJT:2N3904
- removed R1: 1k, symbol Device:R_US
- removed R2, R4: 10k, symbol Device:R_US
- removed R5: 500, symbol Device:R_US
- removed R6: 1M, symbol Device:R_US
- removed V3: 1, symbol Simulation_SPICE:VDC
- added C3, C5: 1, symbol Device:C
- added C4: 100p, symbol Device:C
- added E1: ESOURCE, symbol Simulation_SPICE:ESOURCE
- added R3, R7: 1k, symbol Device:R_US
- added R8: 1M, symbol Device:R_US
- added U1: 4013, symbol 4xxx:4013
- V1: value VSIN -> VWAV
Connections:
- net +9V: now also U1.14 (VDD)
- net 0: now also C4.1, E1.2 (N-), E1.4 (C-), R8.2, U1.4 (R), U1.6 (S), U1.7 (VSS)
- net gain: now also E1.1 (N+), R3.2; no longer B1.1 (N+)
- net in: now also E1.3 (C+)
- net out: now also B1.1 (N+)
- new net: C4.2, C5.2, R7.2
- new net: C3.1, U1.3 (C)
- new net: C3.2, R3.1
- new net: U1.2 (~{Q}), U1.5 (D)
- new net counter: R7.1, U1.1 (Q)
- new net mult: C5.1, R8.1
Other:
- note added: "* .cshunt=10e-15 * .rshunt=10e15 .options chgtol=1e-10 abstol=100u"
- note removed: "* .cshunt=10e-15 * .rshunt=10e15 .options chgtol=1e-11 abstol=10u"

Commit message: high and low octave
Parts:
- added D1, D2: D, symbol Device:D
Connections:
- net 0: now also D1.1 (K), D2.2 (A)
- net clipped: now reaches C3.2, R3.1
- net clipped: now also D1.2 (A), D2.1 (K)
Other:
- note added: ".control tran 20.83u 15 sndparam output.wav 48000 wav24 0.1 0.0 1 sndprint v(out) .endc"
- note removed: ".control tran 20.83u 5 sndparam output.wav 48000 wav24 0.1 0.0 1 sndprint v(out) .endc"
- moved on the sheet: C3, C4, C5, R7, R8, U1A, U1C
