File: octaver/octaver.kicad_sch (KiCad schematic)
At the start: 13 parts, among them U1 4013

Commit message: weh weh I'm kicad and I love crashing weh weh
Parts:
- removed B1: BSOURCE, symbol Simulation_SPICE:BSOURCE
- removed C3: 1, symbol Device:C
- removed C4: 100p, symbol Device:C
- removed D1, D2: D, symbol Device:D
- removed E1: ESOURCE, symbol Simulation_SPICE:ESOURCE
- removed U1: 4013, symbol 4xxx:4013
- removed V1: VWAV, symbol Simulation_SPICE:VSIN
- removed V2: 9, symbol Simulation_SPICE:VDC
- added C1: 1u, Capacitor_SMD:C_0603_1608Metric, symbol Device:C
- added C2: 470n, Capacitor_SMD:C_0603_1608Metric, symbol Device:C
- added C3, C4: 220u, Capacitor_SMD:C_0603_1608Metric, symbol Device:C_Polarized_US
- added C6: 4.7n, Capacitor_SMD:C_0603_1608Metric, symbol Device:C
- added C7: 3.3n, Capacitor_SMD:C_0603_1608Metric, symbol Device:C
- added C8: 22n, Capacitor_SMD:C_0603_1608Metric, symbol Device:C
- added C9: 10u, Capacitor_SMD:C_0603_1608Metric, symbol Device:C
- added D1: On, symbol Device:LED
- added J1: In, Connector_PinHeader_2.54mm:PinHeader_1x02_P2.54mm_Vertical, symbol Connector_Audio:AudioJack2
- added J2: Out, Connector_PinHeader_2.54mm:PinHeader_1x02_P2.54mm_Vertical, symbol Connector_Audio:AudioJack2
- added J3: Power, Connector_PinHeader_2.54mm:PinHeader_1x01_P2.54mm_Vertical, symbol Connector:Jack-DC
- added R1, R16, R2, R20: 1M, Resistor_SMD:R_0201_0603Metric, symbol Device:R_US
- added R10, R14, R4, R9: 10k, Resistor_SMD:R_0201_0603Metric, symbol Device:R_US
- added R11, R17, R6: 100k, Resistor_SMD:R_0201_0603Metric, symbol Device:R_US
- added R12: 1k, Resistor_SMD:R_0201_0603Metric, symbol Device:R_US
- added R13: 12k, Resistor_SMD:R_0201_0603Metric, symbol Device:R_US
- added R15: 1.5k, Resistor_SMD:R_0201_0603Metric, symbol Device:R_US
- added R19: 2k, Resistor_SMD:R_0201_0603Metric, symbol Device:R_US
- added R5: 2.2k, Resistor_SMD:R_0201_0603Metric, symbol Device:R_US
- added RV2: A250k, circuits:Taiss_Potentiometer_vertical, symbol Device:R_Potentiometer_US
- added RV3: B500K, circuits:Taiss_Potentiometer_vertical, symbol Device:R_Potentiometer_US
- added RV5: A100K, circuits:Taiss_Potentiometer_vertical, symbol Device:R_Potentiometer_US
- added RV6: A250K, circuits:Taiss_Potentiometer_vertical, symbol Device:R_Potentiometer_US
- added RV7: A20K, circuits:Taiss_Potentiometer_vertical, symbol Device:R_Potentiometer_US
- added RV8: A1M, circuits:Taiss_Potentiometer_vertical, symbol Device:R_Potentiometer_US
- added SW1: Integrator On, circuits:Adam Tech SW-T3-2B-A-A3-S1, symbol Switch:SW_SPDT
- added SW2: stable / alive, circuits:Adam Tech SW-T3-2B-A-A3-S1, symbol Switch:SW_SPDT
- added SW3: Differentiator On, circuits:Adam Tech SW-T3-2B-A-A3-S1, symbol Switch:SW_SPDT
- added SW4: Octave Lo/Hi, circuits:Adam Tech SW-T3-2B-A-A3-S1, symbol Switch:SW_SPDT
- added SW6: Footswitch, symbol symbols:SW_3PDT_x3
- added U1, U2, U3: TL072, Package_SO:SOIC-8_3.9x4.9mm_P1.27mm, symbol Amplifier_Operational:TL072
- added U5: LM311, Package_SO:SOIC-8_3.9x4.9mm_P1.27mm, symbol Comparator:LM311
- added U6: 40175, Package_SO:SOIC-16_3.9x9.9mm_P1.27mm, symbol 4xxx_IEEE:40175
- added U7: AD633JNZ, footprints:N_8_ADI, symbol AD633:AD633JNZ
- C5: value 1 -> 470n; footprint (none) -> Capacitor_SMD:C_0603_1608Metric
- R3: value 1k -> 12k; footprint (none) -> Resistor_SMD:R_0201_0603Metric
- R7: value 1k -> 100k; footprint (none) -> Resistor_SMD:R_0201_0603Metric
- R8: value 1M -> 1k; footprint (none) -> Resistor_SMD:R_0201_0603Metric
Connections:
- net +9V: now also C3.1, J3.1, R12.2, R6.2, SW6.8 (B), U1.8 (V+), U2.8 (V+), U3.8 (V+), U5.8 (V+), U6.1 (~{R}), U6.16 (Vdd), U7.8 (+VS)
- net at C5.2: now also R10.2, SW3.3 (C), U7.7 (W); no longer R7.2
- net 0: no longer names the net of R8.2
- net 0: now also R9.1, SW2.2 (B)
- net clipped: no longer names the net of R3.1
- net clipped: now also C2.2, R4.2, U2.6 (-)
- net counter renamed GNDPWR
- net GNDPWR: now also C3.2, C4.2, D1.1 (K), J3.2, R1.1, R20.1, U1.4 (V-), U2.4 (V-), U3.4 (V-), U5.1 (GND), U5.4 (V-), U6.8 (Vss), U7.5 (-VS)
- net gain: no longer names the net of R3.2
- net gain: now also RV3.3, SW1.3 (C), U1.1, U1.2 (-)
- net mult: no longer names the net of R8.1
- net mult: now also RV6.1, U2.1, U7.3 (Y1); no longer C5.1
- new net: RV3.2, U3.5 (+)
- new net: R19.2, U3.6 (-), U3.7
- new net: C9.2, RV7.1, U3.1
- new net: R19.1, RV7.2, U3.2 (-)
- new net: C1.1, R2.2, U1.3 (+)
- new net: R11.2, R9.2, SW2.3 (C), U5.2 (+)
- new net: R11.1, R12.1, SW4.3 (C), U5.7, U6.9 (Ck)
- new net: RV2.2, U7.1 (X1)
- new net: C8.1, R16.1, R17.2
- new net: C7.2, R15.1, R16.2
- new net: R5.1, RV6.2, U2.2 (-)
- new net: SW1.2 (B), U2.3 (+)
- new net: D1.2 (A), R14.1
- new net: R14.2, SW6.9 (C)
- new net: C6.1, R13.1, SW3.1 (A), U1.7
- new net: C5.1, C6.2, R10.1, R13.2, U1.6 (-)
- new net: R15.2, RV5.1
- new net: RV5.2, SW3.2 (B)
- new net: C2.1, R4.1, SW1.1 (A), U2.7
- new net: C8.2, RV3.1, RV8.3
- new net: SW4.1 (A), U6.13, U6.14
- new net: SW6.1 (A), SW6.4 (A)
- new net: RV2.1, SW4.2 (B)
- new net GND: C4.1, C7.1, J1.S, J2.S, R17.1, R2.1, R5.2, R6.1, R7.2, RV2.3, RV8.2, U1.5 (+), U2.5 (+), U3.3 (+), U5.3 (-), U7.2 (X2), U7.4 (Y2), U7.6 (Z)
- new net circuit_in: C1.2, R1.2, SW6.3 (C)
- new net circuit_out: C9.1, R20.2, SW6.6 (C)
- new net jack_in: J1.T, SW6.2 (B)
- new net jack_out: J2.T, SW6.5 (B)
- no-connect marks 0 -> 18
Other:
- note added: "Bypass"
- note added: "Cut"
- note added: "Differentiator"
- note added: "Dry/Wet"
- note added: "Integrator"
- note added: "LED"
- note added: "Multiply"
- note added: "Octave"
- note added: "Power"
- note added: "Pre-gain"
- note added: "Tone"
- note added: "Volume"
- note removed: "* .cshunt=10e-15 * .rshunt=10e15 .options chgtol=1e-10 abstol=100u"
- note removed: ".control tran 20.83u 15 sndparam output.wav 48000 wav24 0.1 0.0 1 sndprint v(out) .endc"
- title: (none) -> "the best octave fuzz I've ever played"

Commit message: wow it's like a whole circuit or something
Parts:
- added J4: pot_hp, Connector_PinHeader_2.54mm:PinHeader_1x10_P2.54mm_Vertical, symbol symbols:Conn_01x10_10part
- added J5: sw_hp, Connector_PinHeader_2.54mm:PinHeader_1x10_P2.54mm_Vertical, symbol symbols:Conn_01x10_10part
- added J6: fs_hp, Connector_PinHeader_2.54mm:PinHeader_1x05_P2.54mm_Vertical, symbol symbols:Conn_01x5_5part
- added J7: sw_hp2, Connector_PinHeader_2.54mm:PinHeader_1x05_P2.54mm_Vertical, symbol symbols:Conn_01x5_5part
- added unit 2 of SW6
- added unit 3 of SW6
- C3, C4: footprint Capacitor_SMD:C_0603_1608Metric -> Capacitor_SMD:CP_Elec_8x10.5
- D1: footprint (none) -> LED_THT:LED_D5.0mm
- J1, J2: footprint Connector_PinHeader_2.54mm:PinHeader_1x02_P2.54mm_Vertical -> circuits:mono_jack
- J3: footprint Connector_PinHeader_2.54mm:PinHeader_1x01_P2.54mm_Vertical -> Connector_PinHeader_2.54mm:PinHeader_1x02_P2.54mm_Vertical
- R1, R10, R11, R12, R13, R15, R16, R17, R19, R2, R20, R3, R4, R5, R6, R7, R8, R9: footprint Resistor_SMD:R_0201_0603Metric -> Resistor_SMD:R_0402_1005Metric
- R14: footprint Resistor_SMD:R_0201_0603Metric -> Resistor_THT:R_Axial_DIN0207_L6.3mm_D2.5mm_P10.16mm_Horizontal
- SW6: footprint (none) -> circuits:PBS-24-302_3PDT
- U6: footprint Package_SO:SOIC-16_3.9x9.9mm_P1.27mm -> Package_SO:SOIC-16W_5.3x10.2mm_P1.27mm
Connections:
- net +9V: now also J7.4 (Pin_3); no longer SW6.8 (B)
- net GND: now also J5.10 (Pin_3), J7.3 (Pin_3); no longer C7.1, J1.S, J2.S, R17.1, RV2.3, RV8.2
- net GNDPWR: now also J7.2 (Pin_2); no longer D1.1 (K)
- net circuit_in: now also J7.1 (Pin_3); no longer SW6.3 (C)
- net circuit_out: now also J7.5 (Pin_3); no longer SW6.6 (C)
- net jack_out: now also SW6.5 (B); no longer SW6.5 (B)
- net at U3.5 (+): now also J5.5 (Pin_3); no longer RV3.2
- net at C9.2, U3.1: now also J5.7 (Pin_3); no longer RV7.1
- net at R19.1, U3.2 (-): now also J5.6 (Pin_3); no longer RV7.2
- net at U7.1 (X1): now also J5.8 (Pin_3); no longer RV2.2
- net at R8.1, U2.1, U7.3 (Y1): now also J5.2 (Pin_2); no longer RV6.1
- net at R5.1, U2.2 (-): now also J5.1 (Pin_3); no longer RV6.2
- net at R14.2: now also SW6.9 (C); no longer SW6.9 (C)
- net at SW3.2 (B): now also J5.3 (Pin_3); no longer RV5.2
- net at R3.2, SW1.3 (C), U1.1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: now also J5.4 (Pin_3); no longer RV3.3
- net at SW6.1 (A): now also SW6.4 (A); no longer SW6.4 (A)
- net at RV2.1: now also J4.9 (Pin_3); no longer SW4.2 (B)
- new net: J6.4 (Pin_3), SW6.8 (B)
- new net: J4.4 (Pin_3), RV3.3
- new net: J4.3 (Pin_3), RV5.2
- new net: J4.6 (Pin_3), RV7.2
- new net: J4.2 (Pin_2), RV6.1
- new net: J4.5 (Pin_3), RV3.2
- new net: J4.1 (Pin_3), RV6.2
- new net: J4.8 (Pin_3), RV2.2
- new net: J4.7 (Pin_3), RV7.1
- new net: J5.9 (Pin_3), SW4.2 (B)
- new net: D1.1 (K), J6.2 (Pin_2)
- new net: J6.1 (Pin_3), SW6.3 (C)
- new net: J6.5 (Pin_3), SW6.6 (C)
- new net fsgnd: J1.S, J2.S, J6.3 (Pin_3)
- new net pot_gnd: C7.1, J4.10 (Pin_3), R17.1, RV2.3, RV8.2
Other:
- moved on the sheet: C9, J1, J2, R19, R20, RV2, RV3, RV7, SW3, SW6A, U3A, U3B
