File: octaver/octaver.kicad_pcb (KiCad board)
At the start: 2 copper layers, 16.5 x 16.5 mm, 47 parts, among them J1 In, J2 Out, J3 Power, SW1 Integrator On, SW2 stable / alive, SW3 Differentiator On, SW4 Octave Lo/Hi, U1 TL072, U2 TL072, U3 TL072, U4 TL072, U5 LM311, U6 40175, U7 AD633JNZ

Commit message: wow it's like a whole circuit or something
Parts:
- removed U4: TL072, Package_SO:SOIC-8_3.9x4.9mm_P1.27mm
- added D1: On, LED_THT:LED_D5.0mm, F.Cu at (41.4, 91.9)
- added J4: pot_hp, Connector_PinHeader_2.54mm:PinHeader_1x10_P2.54mm_Vertical, F.Cu at (37.1, 79.8)
- added J5: sw_hp, Connector_PinHeader_2.54mm:PinHeader_1x10_P2.54mm_Vertical, F.Cu at (96.9, 79.8)
- added J6: fs_hp, Connector_PinHeader_2.54mm:PinHeader_1x05_P2.54mm_Vertical, F.Cu at (89.9, 85.9)
- added J7: sw_hp2, Connector_PinHeader_2.54mm:PinHeader_1x05_P2.54mm_Vertical, F.Cu at (145.7, 95.0)
- added R14: 10k, Resistor_THT:R_Axial_DIN0207_L6.3mm_D2.5mm_P10.16mm_Horizontal, F.Cu at (41.5, 98.3)
- added SW6: Footswitch, circuits:PBS-24-302_3PDT, B.Cu at (63.4, 93.6)
- C3, C4: footprint Capacitor_SMD:C_0603_1608Metric -> Capacitor_SMD:CP_Elec_8x10.5
- J1, J2: footprint Connector_PinHeader_2.54mm:PinHeader_1x02_P2.54mm_Vertical -> circuits:mono_jack; moved to B.Cu
- J3: footprint Connector_PinHeader_2.54mm:PinHeader_1x01_P2.54mm_Vertical -> Connector_PinHeader_2.54mm:PinHeader_1x02_P2.54mm_Vertical
- R1, R10, R11, R12, R13, R15, R16, R17, R19, R2, R20, R3, R4, R5, R6, R7, R8, R9: footprint Resistor_SMD:R_0201_0603Metric -> Resistor_SMD:R_0402_1005Metric
- RV2, RV3, RV5, RV6, RV7, RV8, SW1, SW2, SW3, SW4: moved to B.Cu
- U6: footprint Package_SO:SOIC-16_3.9x9.9mm_P1.27mm -> Package_SO:SOIC-16W_5.3x10.2mm_P1.27mm
- moved J1 173.8 mm to (51.1, 85.9), turned to 180 degrees
- moved R3 167.7 mm to (104.4, 75.9), turned to -90 degrees
- moved U2 164.1 mm to (125.7, 73.5), turned to 0 degrees
- moved R5 161.5 mm to (120.9, 72.9), turned to 180 degrees
- moved R4 160.4 mm to (132.3, 73.7), turned to -90 degrees
- moved C2 149.8 mm to (130.8, 73.7), turned to -90 degrees
- moved C9 124.5 mm to (110.5, 61.2), turned to -90 degrees
- moved C4 119.0 mm to (139.2, 29.1), turned to -90 degrees
- moved U3 116.0 mm to (108.6, 67.2)
- moved R19 115.3 mm to (108.0, 73.0), turned to 90 degrees
- moved R6 114.5 mm to (134.6, 22.9), turned to 180 degrees
- moved C3 112.9 mm to (129.5, 29.1)
- moved R7 110.6 mm to (134.6, 34.8), turned to 0 degrees
- moved SW3 110.1 mm to (142.7, 86.5), turned to 180 degrees
- moved R17 108.6 mm to (70.6, 78.7), turned to -90 degrees
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Connections:
- net in renamed circuit_in
- net out renamed circuit_out
- C7 pad 1: GND -> pot_gnd
- C9 pad 2: Net-(C9-Pad2) -> Net-(J5G-Pin_3)
- R17 pad 1: GND -> pot_gnd
- R19 pad 1: Net-(U3A--) -> Net-(J5F-Pin_3)
- R3 pad 2: Net-(SW1-C) -> Net-(J5D-Pin_3)
- R5 pad 1: Net-(U2A--) -> Net-(J5A-Pin_3)
- R8 pad 1: Net-(U7-Y1) -> Net-(J5B-Pin_2)
- RV2 pad 1: Net-(SW4-B) -> Net-(J4I-Pin_3)
- RV2 pad 2: Net-(U7-X1) -> Net-(J4H-Pin_3)
- RV2 pad 3: GND -> pot_gnd
- RV3 pad 2: Net-(U3B-+) -> Net-(J4E-Pin_3)
- RV3 pad 3: Net-(SW1-C) -> Net-(J4D-Pin_3)
- RV5 pad 2: Net-(SW3-B) -> Net-(J4C-Pin_3)
- RV6 pad 1: Net-(U7-Y1) -> Net-(J4B-Pin_2)
- RV6 pad 2: Net-(U2A--) -> Net-(J4A-Pin_3)
- RV7 pad 1: Net-(C9-Pad2) -> Net-(J4G-Pin_3)
- RV7 pad 2: Net-(U3A--) -> Net-(J4F-Pin_3)
- RV8 pad 2: GND -> pot_gnd
- SW1 pad 3: Net-(SW1-C) -> Net-(J5D-Pin_3)
- SW3 pad 2: Net-(SW3-B) -> Net-(J5C-Pin_3)
- SW4 pad 2: Net-(SW4-B) -> Net-(J5I-Pin_3)
- U1 pad 1: Net-(SW1-C) -> Net-(J5D-Pin_3)
- U1 pad 2: Net-(SW1-C) -> Net-(J5D-Pin_3)
- U2 pad 1: Net-(U7-Y1) -> Net-(J5B-Pin_2)
- U2 pad 2: Net-(U2A--) -> Net-(J5A-Pin_3)
- U3 pad 1: Net-(C9-Pad2) -> Net-(J5G-Pin_3)
- U3 pad 2: Net-(U3A--) -> Net-(J5F-Pin_3)
- U3 pad 5: Net-(U3B-+) -> Net-(J5E-Pin_3)
- U7 pad 1: Net-(U7-X1) -> Net-(J5H-Pin_3)
- U7 pad 3: Net-(U7-Y1) -> Net-(J5B-Pin_2)
Routing:
- net GNDPWR: track 0.00 -> 185.7 mm, vias 0 -> 15
- net +9V: track 0.00 -> 174.2 mm, vias 0 -> 7
- net Net-(J5B-Pin_2): track 0.00 -> 79.7 mm, vias 0 -> 4
- net Net-(J4B-Pin_2): track 0.00 -> 73.0 mm
- net Net-(J4A-Pin_3): track 0.00 -> 71.2 mm
- net Net-(J5D-Pin_3): track 0.00 -> 60.5 mm, vias 0 -> 3
- net Net-(D1-K): track 0.00 -> 57.6 mm
- net circuit_out: track 0.00 -> 51.4 mm, vias 0 -> 2
- net Net-(J5C-Pin_3): track 0.00 -> 47.2 mm, vias 0 -> 1
- net Net-(J5H-Pin_3): track 0.00 -> 46.5 mm
- net Net-(J4C-Pin_3): track 0.00 -> 42.5 mm
- net Net-(J4I-Pin_3): track 0.00 -> 41.4 mm
- net Net-(SW1-A): track 0.00 -> 37.7 mm, vias 0 -> 2
- net Net-(J4H-Pin_3): track 0.00 -> 37.5 mm
- net Net-(J4F-Pin_3): track 0.00 -> 37.1 mm
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- added copper zone on B.Cu, net /fsgnd
- added copper zone on F.Cu, net /fsgnd
- added copper zone on B.Cu, net GND
- added copper zone on F.Cu, net GND
- added copper zone on B.Cu, net pot_gnd
- added copper zone on F.Cu, net pot_gnd
Other:
- board size 16.5 x 16.5 mm -> 119.1 x 83.8 mm
- board text added: "+"
- board text added: "-"
