File: src/fridge/board/devboard/devboard.kicad_sch (KiCad schematic)
At the start: 11 parts, among them SW1 RotaryEncoder_Switch, U1 CD4051B, U2 IS31FL3731-QF, U3 CD4051B, U4 CD4051B, U5 CD4051B, U6 CD4051B, U7 CD4051B, U8 TL072

Commit message: create a dev board
add most switches, LED matrix A

attach LED controller, output amp

adjust output buffer & run ERC

re-annotate schematic

start work on part choice

draw encoder footprint

use PJ-037A power jack

add audio jacks and 4P4T switch

update PCB and set BOM/POS

run ERC

start routingggggggg

route LED connections for buttons

think about control layout

most analog routing, some address

pour copper on board

wip

wip

mostly finish routing

maybe actually finish routing

run DRC

stitch vias, correct power jack

beef up GNDA and add housing lug

start addressing review comments

re-assign JLC #s

add mounting holes, remove unpopulated parts from BOM

get devboard ready for fab

add "quote"

production files!
Parts:
- removed D1: LED_ABGR, symbol Device:LED_ABGR
- removed SW1: RotaryEncoder_Switch, symbol Device:RotaryEncoder_Switch
- removed U3, U7: CD4051B, symbol Analog_Switch:CD4051B
- added C1, C2: 33n, Capacitor_SMD:C_0603_1608Metric, symbol Device:C
- added C3, C4, C6, C7: 4.7u, Capacitor_SMD:C_0603_1608Metric, symbol Device:C
- added C5: 2.2u, Capacitor_SMD:C_0603_1608Metric, symbol Device:C
- added C8: 220n, Capacitor_SMD:C_0603_1608Metric, symbol Device:C
- added C9: 100n, Capacitor_SMD:C_0603_1608Metric, symbol Device:C
- added D1, D10, D11, D12, D13, D14, D15, D16, D17, D18, D19, D2, D20, D21, D22, D23, D24, D25, D26, D27, D28, D29, D3, D30, D31, D32, D33, D34, D35, D36, D37, D38, D39, D4, D40, D41, D42, D43, D44, D45, D46, D47, D48, D5, D6, D7, D8, D9: LED_RGB, devboard:E6C1615RGBC3UDA-A01, symbol Device:LED_RGB
- added H1, H2, H3, H4: MountingHole, MountingHole:MountingHole_3.2mm_M3, symbol Mechanical:MountingHole
- added J1, J2: SN37A14B, devboard:SWITCHCRAFT_SN37A14B, symbol SN37A14B:SN37A14B
- added J3: PJ-037A, devboard:CUI_PJ-037A, symbol PJ-037A:PJ-037A
- added JP1: Jumper_2_Bridged, Jumper:SolderJumper-2_P1.3mm_Bridged_RoundedPad1.0x1.5mm, symbol Jumper:Jumper_2_Bridged
- added N1: Housing_Pad, TestPoint:TestPoint_THTPad_4.0x4.0mm_Drill2.0mm, symbol Mechanical:Housing_Pad
- added R1, R2, R5, R6, R7, R9: 1M, Resistor_SMD:R_0603_1608Metric, symbol Device:R_US
- added R10, R8: 100, Resistor_SMD:R_0603_1608Metric, symbol Device:R_US
- added R11, R13, R14: 4.7k, Resistor_SMD:R_0603_1608Metric, symbol Device:R_US
- added R12: 20k, Resistor_SMD:R_0603_1608Metric, symbol Device:R_US
- added R15: 100k, Resistor_SMD:R_0603_1608Metric, symbol Device:R_US
- added R3, R4: 1k, Resistor_SMD:R_0603_1608Metric, symbol Device:R_US
- added RV1, RV2: 100k, devboard:Taiss_Potentiometer, symbol Device:R_Potentiometer_US
- added SW1: EG4208A, devboard:SWITCH12_EG4208A_EWI, symbol EG4208A:EG4208A
- added SW10, SW11, SW12, SW13, SW14, SW15, SW16, SW17, SW2, SW3, SW4, SW5, SW6, SW7, SW8, SW9: RotaryEncoder_Switch, devboard:Encoder_PEC12R-3225F-S0024, symbol Device:RotaryEncoder_Switch
- added SW18, SW19, SW20, SW21, SW22, SW23, SW24, SW25, SW26, SW27, SW28, SW29, SW30, SW31, SW32, SW33: SW_Push, devboard:Button_C4B1802110, symbol Switch:SW_Push
- added TP1, TP10, TP11, TP12, TP13, TP14, TP15, TP16, TP17, TP18, TP19, TP2, TP20, TP21, TP22, TP23, TP3, TP4, TP5, TP6, TP7, TP8, TP9: TestPoint, TestPoint:TestPoint_Pad_1.0x1.0mm, symbol Connector:TestPoint
- added U1, U10, U2, U8: CD4051B, Package_SO:SOIC-16_3.9x9.9mm_P1.27mm, symbol Analog_Switch:CD4051B
- U3: renamed from U8; footprint (none) -> Package_SO:SO-8_3.9x4.9mm_P1.27mm
- U4, U5, U6: footprint (none) -> Package_SO:SOIC-16_3.9x9.9mm_P1.27mm
- U9: renamed from U1; footprint (none) -> Package_SO:SOIC-16_3.9x9.9mm_P1.27mm
- renumbered U2 to U7
Connections:
- net at U4.1 (X4): now also SW6.S1
- net A1: now reaches U4.10 (B)
- net A1: now also A1.2 (SD_DATA_3), U5.10 (B), U6.10 (B), U9.10 (B), U1.10 (B), U10.10 (B), U2.10 (B), U8.10 (B)
- net A0: now reaches U4.11 (A)
- net A0: now also A1.1 (USB_ID), U5.11 (A), U6.11 (A), U9.11 (A), U1.11 (A), U10.11 (A), U2.11 (A), U8.11 (A)
- net at U4.12 (X3): now also SW5.S1
- net at U4.13 (X0): now also SW2.S1
- net at U4.14 (X1): now also SW3.S1
- net at U4.15 (X2): now also SW4.S1
- net +3V3: now reaches U4.16 (VDD)
- net +3V3: now also A1.38 (3V3_D), U5.16 (VDD), U6.16 (VDD), U7.2 (VCC), U9.16 (VDD), R11.1, R13.1, R14.1, U1.16 (VDD), U10.16 (VDD), U2.16 (VDD), U8.16 (VDD)
- net at U4.2 (X6): now also SW8.S1
- net KNOB_S0: now reaches U4.3 (X)
- net KNOB_S0: now also A1.10 (SPI1_POCI)
- net at U4.4 (X7): now also SW9.S1
- net at U4.5 (X5): now also SW7.S1
- net GND: now reaches U4.6 (INH)
- net GND: now also A1.40 (DGND), U3.4 (V-), U4.7 (VEE), U4.8 (VSS), U5.6 (INH), U5.7 (VEE), U5.8 (VSS), U6.6 (INH), U6.7 (VEE), U6.8 (VSS), U7.18 (AD), U7.29 (GND), U7.5 (GND), U9.6 (INH), U9.7 (VEE), U9.8 (VSS), C9.2, J3.1, JP1.1 (A), R12.2, R15.2, R6.1, SW10.C, SW10.S2, SW11.C, SW11.S2, SW12.C, SW12.S2, SW13.C, SW13.S2, SW14.C, SW14.S2, SW15.C, SW15.S2, SW16.C, SW16.S2, SW17.C, SW17.S2, SW18.2, SW19.2, SW2.C, SW2.S2, SW20.2, SW21.2, SW22.2, SW23.2, SW24.2, SW25.2, SW26.2, SW27.2, SW28.2, SW29.2, SW3.C, SW3.S2, SW30.2, SW31.2, SW32.2, SW33.2, SW4.C, SW4.S2, SW5.C, SW5.S2, SW6.C, SW6.S2, SW7.C, SW7.S2, SW8.C, SW8.S2, SW9.C, SW9.S2, U1.6 (INH), U1.7 (VEE), U1.8 (VSS), U10.6 (INH), U10.7 (VEE), U10.8 (VSS), U2.6 (INH), U2.7 (VEE), U2.8 (VSS), U8.6 (INH), U8.7 (VEE), U8.8 (VSS)
- net A2: now reaches U4.9 (C)
- net A2: now also A1.3 (SD_DATA_2), U5.9 (C), U6.9 (C), U9.9 (C), U1.9 (C), U10.9 (C), U2.9 (C), U8.9 (C)
- net at U5.1 (X4): now also SW14.A
- net at U5.12 (X3): now also SW13.A
- net at U5.13 (X0): now also SW10.A
- net at U5.14 (X1): now also SW11.A
- net at U5.15 (X2): now also SW12.A
- net at U5.2 (X6): now also SW16.A
- net KNOB_A1: now reaches U5.3 (X)
- net KNOB_A1: now also A1.8 (SPI1_CS)
- net at U5.4 (X7): now also SW17.A
- net at U5.5 (X5): now also SW15.A
- net AMP_REF: now reaches U3.5 (+)
- net AMP_REF: now also U3.3 (+), C5.2, R5.1, R6.2
- net at U3.6 (-): now also R4.1, RV2.2
- net at U3.7: now also C7.2, RV2.3
- net at U9.1 (X4): now also SW22.1
- net at U9.12 (X3): now also SW21.1
- net at U9.13 (X0): now also SW18.1
- net at U9.14 (X1): now also SW19.1
- net at U9.15 (X2): now also SW20.1
- net at U9.2 (X6): now also SW24.1
- net SW0: now reaches U9.3 (X)
- net SW0: now also A1.4 (SD_DATA_1)
- net at U9.4 (X7): now also SW25.1
- net at U9.5 (X5): now also SW23.1
- net VCC: now reaches U3.8 (V+)
- net VCC: now also A1.39 (VIN), J3.2, R5.2
- net CA9: now reaches U7.1 (CA9)
- net CA9: now also D15.3 (BK), D21.3 (BK), D27.3 (BK), D3.3 (BK), D33.3 (BK), D39.3 (BK), D43.4 (BA), D43.5 (GA), D43.6 (RA), D44.4 (BA), D44.5 (GA), D44.6 (RA), D45.3 (BK), D45.5 (GA), D45.6 (RA), D9.3 (BK)
- net CB4: now reaches U7.10 (CB4)
- net CB4: now also D11.1 (RK), D16.4 (BA), D16.5 (GA), D16.6 (RA), D17.1 (RK), D23.1 (RK), D23.4 (BA), D23.5 (GA), D24.4 (BA), D24.5 (GA), D24.6 (RA), D29.1 (RK), D35.1 (RK), D41.1 (RK), D47.1 (RK), D5.1 (RK)
- net CB5: now reaches U7.11 (CB5)
- net CB5: now also D11.2 (GK), D17.2 (GK), D22.4 (BA), D22.5 (GA), D22.6 (RA), D23.2 (GK), D23.6 (RA), D29.2 (GK), D29.4 (BA), D30.4 (BA), D30.5 (GA), D30.6 (RA), D35.2 (GK), D41.2 (GK), D47.2 (GK), D5.2 (GK)
- net CB6: now reaches U7.12 (CB6)
- net CB6: now also D11.3 (BK), D17.3 (BK), D23.3 (BK), D28.4 (BA), D28.5 (GA), D28.6 (RA), D29.3 (BK), D29.5 (GA), D29.6 (RA), D35.3 (BK), D36.4 (BA), D36.5 (GA), D36.6 (RA), D41.3 (BK), D47.3 (BK), D5.3 (BK)
- net CB7: now reaches U7.13 (CB7)
- net CB7: now also D12.1 (RK), D18.1 (RK), D24.1 (RK), D30.1 (RK), D34.4 (BA), D34.5 (GA), D34.6 (RA), D35.4 (BA), D35.5 (GA), D35.6 (RA), D36.1 (RK), D42.1 (RK), D42.4 (BA), D42.5 (GA), D48.1 (RK), D6.1 (RK)
- net CB8: now reaches U7.14 (CB8)
- net CB8: now also D12.2 (GK), D18.2 (GK), D24.2 (GK), D30.2 (GK), D36.2 (GK), D40.4 (BA), D40.5 (GA), D40.6 (RA), D41.4 (BA), D41.5 (GA), D41.6 (RA), D42.2 (GK), D42.6 (RA), D48.2 (GK), D48.4 (BA), D6.2 (GK)
- net CB9: now reaches U7.15 (CB9)
- net CB9: now also D12.3 (BK), D18.3 (BK), D24.3 (BK), D30.3 (BK), D36.3 (BK), D42.3 (BK), D46.4 (BA), D46.5 (GA), D46.6 (RA), D47.4 (BA), D47.5 (GA), D47.6 (RA), D48.3 (BK), D48.5 (GA), D48.6 (RA), D6.3 (BK)
- net at U7.16 (C_FILT): now also C9.1
- net at U7.17 (IN): now also C8.2
- net LED_SDA: now reaches U7.19 (SDA)
- net LED_SDA: now also A1.13 (I2C1_SDA), R11.2
- net LED_SCL: now reaches U7.20 (SCL)
- net LED_SCL: now also A1.12 (I2C1_SCL), R13.2
- net CA1: now reaches U7.21 (CA1)
- net CA1: now also D1.1 (RK), D1.4 (BA), D1.5 (GA), D13.1 (RK), D19.1 (RK), D2.4 (BA), D2.5 (GA), D2.6 (RA), D25.1 (RK), D3.4 (BA), D3.5 (GA), D3.6 (RA), D31.1 (RK), D37.1 (RK), D43.1 (RK), D7.1 (RK)
- net CA2: now reaches U7.22 (CA2)
- net CA2: now also D1.2 (GK), D1.6 (RA), D13.2 (GK), D19.2 (GK), D25.2 (GK), D31.2 (GK), D37.2 (GK), D43.2 (GK), D7.2 (GK), D7.4 (BA), D8.4 (BA), D8.5 (GA), D8.6 (RA), D9.4 (BA), D9.5 (GA), D9.6 (RA)
- net CA3: now reaches U7.23 (CA3)
- net CA3: now also D1.3 (BK), D13.3 (BK), D14.4 (BA), D14.5 (GA), D14.6 (RA), D15.4 (BA), D15.5 (GA), D15.6 (RA), D19.3 (BK), D25.3 (BK), D31.3 (BK), D37.3 (BK), D43.3 (BK), D7.3 (BK), D7.5 (GA), D7.6 (RA)
- net CA4: now reaches U7.24 (CA4)
- net CA4: now also D13.4 (BA), D13.5 (GA), D13.6 (RA), D14.1 (RK), D2.1 (RK), D20.1 (RK), D20.4 (BA), D20.5 (GA), D21.4 (BA), D21.5 (GA), D21.6 (RA), D26.1 (RK), D32.1 (RK), D38.1 (RK), D44.1 (RK), D8.1 (RK)
- net CA5: now reaches U7.25 (CA5)
- net CA5: now also D14.2 (GK), D19.4 (BA), D19.5 (GA), D19.6 (RA), D2.2 (GK), D20.2 (GK), D20.6 (RA), D26.2 (GK), D26.4 (BA), D27.4 (BA), D27.5 (GA), D27.6 (RA), D32.2 (GK), D38.2 (GK), D44.2 (GK), D8.2 (GK)
- net CA6: now reaches U7.26 (CA6)
- net CA6: now also D14.3 (BK), D2.3 (BK), D20.3 (BK), D25.4 (BA), D25.5 (GA), D25.6 (RA), D26.3 (BK), D26.5 (GA), D26.6 (RA), D32.3 (BK), D33.4 (BA), D33.5 (GA), D33.6 (RA), D38.3 (BK), D44.3 (BK), D8.3 (BK)
- net CA7: now reaches U7.27 (CA7)
- net CA7: now also D15.1 (RK), D21.1 (RK), D27.1 (RK), D3.1 (RK), D31.4 (BA), D31.5 (GA), D31.6 (RA), D32.4 (BA), D32.5 (GA), D32.6 (RA), D33.1 (RK), D39.1 (RK), D39.4 (BA), D39.5 (GA), D45.1 (RK), D9.1 (RK)
- net CA8: now reaches U7.28 (CA8)
- net CA8: now also D15.2 (GK), D21.2 (GK), D27.2 (GK), D3.2 (GK), D33.2 (GK), D37.4 (BA), D37.5 (GA), D37.6 (RA), D38.4 (BA), D38.5 (GA), D38.6 (RA), D39.2 (GK), D39.6 (RA), D45.2 (GK), D45.4 (BA), D9.2 (GK)
- net ~{LED_SDB}: now reaches U7.3 (~{SDB})
- net ~{LED_SDB}: now also A1.15 (USART1_RX), R15.1
- net ~{LED_INTB}: now reaches U7.4 (~{INTB})
- net ~{LED_INTB}: now also A1.14 (USART1_TX), R14.2
- net at U7.6 (R_EXT): now also R12.1
- net CB1: now reaches U7.7 (CB1)
- net CB1: now also D10.1 (RK), D16.1 (RK), D22.1 (RK), D28.1 (RK), D34.1 (RK), D4.1 (RK), D4.4 (BA), D4.5 (GA), D40.1 (RK), D46.1 (RK), D5.4 (BA), D5.5 (GA), D5.6 (RA), D6.4 (BA), D6.5 (GA), D6.6 (RA)
- net CB2: now reaches U7.8 (CB2)
- net CB2: now also D10.2 (GK), D10.4 (BA), D11.4 (BA), D11.5 (GA), D11.6 (RA), D12.4 (BA), D12.5 (GA), D12.6 (RA), D16.2 (GK), D22.2 (GK), D28.2 (GK), D34.2 (GK), D4.2 (GK), D4.6 (RA), D40.2 (GK), D46.2 (GK)
- net CB3: now reaches U7.9 (CB3)
- net CB3: now also D10.3 (BK), D10.5 (GA), D10.6 (RA), D16.3 (BK), D17.4 (BA), D17.5 (GA), D17.6 (RA), D18.4 (BA), D18.5 (GA), D18.6 (RA), D22.3 (BK), D28.3 (BK), D34.3 (BK), D4.3 (BK), D40.3 (BK), D46.3 (BK)
- net at U3.1: now also C6.2, RV1.3
- net at U3.2 (-): now also R3.1, RV1.2
- net at U6.1 (X4): now also SW14.B
- net at U6.12 (X3): now also SW13.B
- net at U6.13 (X0): now also SW10.B
- net at U6.14 (X1): now also SW11.B
- net at U6.15 (X2): now also SW12.B
- net at U6.2 (X6): now also SW16.B
- net KNOB_B1: now reaches U6.3 (X)
- net KNOB_B1: now also A1.9 (SPI1_SCK)
- net at U6.4 (X7): now also SW17.B
- net at U6.5 (X5): now also SW15.B
- net KNOB_S1: now reaches A1.11 (SPI1_PICO)
- net KNOB_S1: now also U8.3 (X)
- net AUDIO_IN_1: now reaches A1.16 (AUDIO_IN_1)
- net AUDIO_IN_1: now also J1.T, TP6.1
- net AUDIO_IN_2: now reaches A1.17 (AUDIO_IN_2)
- net AUDIO_IN_2: now also J1.R, TP5.1
- net AUDIO_OUT_1: now reaches A1.18 (AUDIO_OUT_1)
- net AUDIO_OUT_1: now also C1.2, SW1.8
- net AUDIO_OUT_2: now reaches A1.19 (AUDIO_OUT_2)
- net AUDIO_OUT_2: now also C2.2, SW1.11
- net GNDA: now reaches A1.20 (AGND)
- net GNDA: now also C1.1, C2.1, C5.1, J1.S, J2.S, JP1.2 (B), N1.1 (PAD), R1.2, R2.2, R7.2, R9.2
- net +3V3_A: now reaches A1.21 (3V3_A)
- net at A1.22 (ADC_0): now also TP9.1
- net at A1.23 (ADC_1): now also TP10.1
- net at A1.24 (ADC_2): now also TP11.1
- net at A1.25 (ADC_3): now also TP12.1
- net at A1.26 (ADC_4): now also TP13.1
- net at A1.27 (ADC_5): now also TP14.1
- net at A1.28 (ADC_6): now also TP15.1
- net at A1.29 (DAC_OUT2): now also TP16.1
- net LED_AUDIO: now reaches A1.30 (DAC_OUT1)
- net LED_AUDIO: now also C8.1
- net at A1.31 (SAI2_MCLK): now also TP17.1
- net at A1.32 (SAI2_SD_B): now also TP18.1
- net at A1.33 (SAI2_SD_A): now also TP19.1
- net at A1.34 (SAI2_FS): now also TP20.1
- net at A1.35 (SAI2_SCK): now also TP21.1
- net at A1.36 (USB_D_-): now also TP22.1
- net at A1.37 (USB_D_+): now also TP23.1
- net SW1: now reaches A1.5 (SD_DATA_0)
- net SW1: now also U10.3 (X)
- net KNOB_A0: now reaches A1.6 (SD_CMD)
- net KNOB_A0: now also U1.3 (X)
- net KNOB_B0: now reaches A1.7 (SD_CLK)
- net KNOB_B0: now also U2.3 (X)
- new net: SW8.A, U1.2 (X6)
- new net: SW8.B, U2.2 (X6)
- new net: J2.TB, TP4.1
- new net: C6.1, R10.1, R7.1
- new net: SW33.1, U10.4 (X7)
- new net: R10.2, SW1.3
- new net: SW4.A, U1.15 (X2)
- new net: SW4.B, U2.15 (X2)
- new net: R8.1, SW1.6
- new net: C7.1, R8.2, R9.1
- new net: C3.2, R1.1, SW1.9
- new net: C3.1, R3.2
- new net: SW5.A, U1.12 (X3)
- new net: SW5.B, U2.12 (X3)
- new net: SW15.S1, U8.5 (X5)
- new net: J1.RB, TP1.1
- new net: J1.TB, TP2.1
- new net: SW31.1, U10.5 (X5)
- new net: SW12.S1, U8.15 (X2)
- new net: SW3.A, U1.14 (X1)
- new net: SW3.B, U2.14 (X1)
- new net: SW14.S1, U8.1 (X4)
- new net: SW30.1, U10.1 (X4)
- new net: C4.1, R2.1, SW1.12
- new net: SW27.1, U10.14 (X1)
- new net: SW29.1, U10.12 (X3)
- new net: SW26.1, U10.13 (X0)
- new net: SW28.1, U10.15 (X2)
- new net: SW32.1, U10.2 (X6)
- new net: C4.2, R4.2
- new net: SW1.1, SW1.7
- new net: SW1.10, SW1.4
- new net: SW6.A, U1.1 (X4)
- new net: SW6.B, U2.1 (X4)
- new net: SW17.S1, U8.4 (X7)
- new net: SW2.A, U1.13 (X0)
- new net: SW2.B, U2.13 (X0)
- new net: SW9.B, U2.4 (X7)
- new net: SW7.B, U2.5 (X5)
- new net: J2.RB, TP3.1
- new net: SW9.A, U1.4 (X7)
- new net: SW7.A, U1.5 (X5)
- new net: SW13.S1, U8.12 (X3)
- new net: SW10.S1, U8.13 (X0)
- new net: SW11.S1, U8.14 (X1)
- new net: SW16.S1, U8.2 (X6)
- new net AUDIO_OUT_1_AMP: J2.T, SW1.2, TP8.1
- new net AUDIO_OUT_2_AMP: J2.R, SW1.5, TP7.1
- no-connect marks 0 -> 2
Other:
- note added: "i (nausicaa) am 100% sure that, given a capacitively-coupled input, the input to this inverting amplifier will self-reference to AMP_REF."
- note added: "the daisy seed has 100 Ω of output impedance, so a 33 nF capacitor here gives a lowpass knee of about 48 kHz."
- note added: "this switch cuts out the output audio amplifiers. since the TL072s run from VCC (at least 9 V), they won't get power if we're running this pedal from USB. flipping this switch allows us to use the daisy's audio out lines directly in that case."
- note added: "~1.1 s time constant, will take around 2 s to start up fully"
- title: (none) -> daisy devboard
- moved on the sheet: A1, U3A, U3B, U3C, U7, U9
