File: hardware/projects/stud/stud.kicad_pcb (KiCad board)
At the start: 4 copper layers, 7 parts, among them IC1 R7KA8M2JFLCAC#UC0, IC2 IS42S32160F-7BLI, J1 USB_C_Receptacle_USB2.0_16P, U1 TPS629210DRLR, U2 TAC5242, Y1 X1G0044510004

Commit message: choose some parts and start routing
Parts:
- removed J1: USB_C_Receptacle_USB2.0_16P, Connector_USB:USB_C_Receptacle_G-Switch_GT-USB-7010ASV
- removed MICRO_SD1: TF-01A, vendor:TF-01A
- removed U1: TPS629210DRLR, vendor:SOT50P160X60-8N
- removed U2: TAC5242, custom:Texas_VQFN-24-1EP_4x4mm_P0.5mm_EP2.1x2.1mm_ThermalVias_CornerPad
- removed Y1: X1G0044510004, custom:SG5032CAN
- moved IC2 0.70 mm to (122.6, 109.4)
- moved IC1 0.20 mm to (134.7, 109.4)
Connections:
- IC1 pad A12: unconnected-(IC1-P309-PadA12) -> Net-(IC1-P309)
- IC1 pad A13: unconnected-(IC1-P906-PadA13) -> Net-(IC1-P906)
- IC1 pad A15: unconnected-(IC1-P907-PadA15) -> Net-(IC1-P907)
- IC1 pad A16: unconnected-(IC1-P904-PadA16) -> Net-(IC1-P904)
- IC1 pad B12: unconnected-(IC1-P311-PadB12) -> Net-(IC1-P311)
- IC1 pad B13: unconnected-(IC1-P908-PadB13) -> Net-(IC1-P908)
- IC1 pad B14: unconnected-(IC1-P909-PadB14) -> Net-(IC1-P909)
- IC1 pad B6: unconnected-(IC1-P303-PadB6) -> Net-(IC1-P303)
- IC1 pad C13: unconnected-(IC1-P312-PadC13) -> Net-(IC1-P312)
- IC1 pad C17: unconnected-(IC1-PD06-PadC17) -> Net-(IC1-PD06)
- IC1 pad C6: unconnected-(IC1-P210/T_MS/S_WDIO-PadC6) -> SWDIO
- IC1 pad C7: unconnected-(IC1-P208/T_DI-PadC7) -> +3V3
- IC1 pad D5: unconnected-(IC1-RES-PadD5) -> ~{RESET}
- IC1 pad D6: unconnected-(IC1-P211/T_CK/S_WCLK-PadD6) -> SWCLK
- IC1 pad E16: unconnected-(IC1-PB00-PadE16) -> Net-(IC1-PB00)
- IC1 pad E7: unconnected-(IC1-P209/TDO-PadE7) -> SWO
- IC1 pad F16: unconnected-(IC1-P707-PadF16) -> SSI_ERROR
- IC1 pad F17: unconnected-(IC1-P705-PadF17) -> Net-(IC1-P705)
- IC1 pad F9: unconnected-(IC1-VCL3-PadF9) -> +0V9
- IC1 pad J11: unconnected-(IC1-VCL2-PadJ11) -> +0V9
- IC1 pad K13: unconnected-(IC1-P410-PadK13) -> Net-(IC1-P410)
- IC1 pad L10: unconnected-(IC1-VCL10-PadL10) -> +0V9
- IC1 pad N1: unconnected-(IC1-P605-PadN1) -> Net-(IC1-P605)
- IC1 pad N15: unconnected-(IC1-P711-PadN15) -> Net-(IC1-P711)
- IC1 pad N16: unconnected-(IC1-P713-PadN16) -> Net-(IC1-P713)
- IC1 pad P1: unconnected-(IC1-P603-PadP1) -> Net-(IC1-P603)
- IC1 pad P11: unconnected-(IC1-P009-PadP11) -> Net-(IC1-P009)
- IC1 pad P13: unconnected-(IC1-P512-PadP13) -> Net-(IC1-P512)
- IC1 pad P15: unconnected-(IC1-P515-PadP15) -> Net-(IC1-P515)
- IC1 pad P16: unconnected-(IC1-P709-PadP16) -> Net-(IC1-P709)
- IC1 pad P2: unconnected-(IC1-P602-PadP2) -> Net-(IC1-P602)
- IC1 pad R11: unconnected-(IC1-P005-PadR11) -> Net-(IC1-P005)
- IC1 pad R12: unconnected-(IC1-P003-PadR12) -> Net-(IC1-P003)
- IC1 pad R14: unconnected-(IC1-P514-PadR14) -> Net-(IC1-P514)
- IC1 pad R16: unconnected-(IC1-P409-PadR16) -> Net-(IC1-P409)
- IC1 pad R17: unconnected-(IC1-P407-PadR17) -> Net-(IC1-P407)
- IC1 pad T1: unconnected-(IC1-P205-PadT1) -> Net-(IC1-P205)
- IC1 pad T12: unconnected-(IC1-P007-PadT12) -> Net-(IC1-P007)
- IC1 pad T13: unconnected-(IC1-P001-PadT13) -> Net-(IC1-P001)
- IC1 pad T15: unconnected-(IC1-P715-PadT15) -> Net-(IC1-P715)
- IC1 pad T2: unconnected-(IC1-P203-PadT2) -> Net-(IC1-P203)
- IC1 pad T3: unconnected-(IC1-P313-PadT3) -> Net-(IC1-P313)
- IC1 pad T8: unconnected-(IC1-P014-PadT8) -> Net-(IC1-P014)
- IC1 pad U1: unconnected-(IC1-P204-PadU1) -> Net-(IC1-P204)
- IC1 pad U11: unconnected-(IC1-P008-PadU11) -> Net-(IC1-P008)
- IC1 pad U12: unconnected-(IC1-P006-PadU12) -> Net-(IC1-P006)
- IC1 pad U13: unconnected-(IC1-P000-PadU13) -> Net-(IC1-P000)
- IC1 pad U14: unconnected-(IC1-P002-PadU14) -> Net-(IC1-P002)
- IC1 pad U15: unconnected-(IC1-P511-PadU15) -> Net-(IC1-P511)
- IC1 pad U2: unconnected-(IC1-P202-PadU2) -> Net-(IC1-P202)
- IC1 pad U6: unconnected-(IC1-P100-PadU6) -> Net-(IC1-P100)
- IC1 pad U8: unconnected-(IC1-P015-PadU8) -> Net-(IC1-P015)
Routing:
- net DQ6: track 0.00 -> 17.0 mm, vias 0 -> 2
- net DQ23: track 0.00 -> 16.0 mm, vias 0 -> 2
- net DQ21: track 0.00 -> 15.8 mm, vias 0 -> 2
- net DQ19: track 0.00 -> 15.6 mm, vias 0 -> 2
- net DQ20: track 0.00 -> 15.5 mm, vias 0 -> 2
- net DQ3: track 0.00 -> 15.2 mm, vias 0 -> 2
- net DQ2: track 0.00 -> 14.9 mm, vias 0 -> 2
- net DQ5: track 0.00 -> 14.1 mm, vias 0 -> 2
- net DQ16: track 0.00 -> 14.1 mm, vias 0 -> 2
- net DQ18: track 0.00 -> 14.0 mm, vias 0 -> 2
- net DQ22: track 0.00 -> 13.4 mm, vias 0 -> 2
- net DQ0: track 0.00 -> 13.4 mm, vias 0 -> 2
- net DQ17: track 0.00 -> 13.0 mm, vias 0 -> 2
- net DQ4: track 0.00 -> 12.4 mm, vias 0 -> 2
- net DQ7: track 0.00 -> 12.2 mm, vias 0 -> 2
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