File: hardware/projects/stud/stud.kicad_sch (KiCad schematic)
At the start: 122 parts, among them IC1 R7KA8M2JFLCAC#UC0, IC2 IS42S32160F-7BLI, J1 USB_C_Receptacle_USB2.0_16P, J10 SCL1_A, J11 SDA1_A, J12 SCL2_B, J13 SDA2_B, J14 RSPCKA_A, J15 MOSIA_A, J16 MISOA_A, J17 SSLA0_A, J18 CTX0, J19 CRX0, J2 DAC0, J20 GTIOC13A, J21 GTIOC13B, J22 GTIOC12A, J23 GTIOC12B, J24 GTIOC11B, J25 GTIOC2A, J26 GTIOC8A, J27 GTIOC8B, J28 TXD0_B, J29 RXD0_B, J3 ADC1_8, J30 VCOUT, J31 IVREF1, J32 ADC1_1, J33 ADC1_3, J34 ADC1_5, J35 ADC1_7, J36 ADTRG0, J37 PDMCLK2, J38 PDMDAT2, J39 P205, J4 DAC1, J40 P303, J41 P709, J42 P711, J43 P713, J44 P715, J5 ADC1_6, J6 ADC1_0, J7 ADC1_2, J8 SCL0_A, J9 SDA0_A, U1 TPS629210DRLR, U2 TAC5242, Y1 X1G0044510004

Commit message: hook up a debug port, audio io, wall off unused
Parts:
- added J45: Conn_ARM_SWD_TagConnect_TC2030-NL, Connector:Tag-Connect_TC2030-IDC-NL_2x03_P1.27mm_Vertical, symbol Connector:Conn_ARM_SWD_TagConnect_TC2030-NL
- added J46: +9V, custom:Connector_01x01_CastellatedEdge, symbol custom:Connector_01x01_CastellatedEdge
- added J47: VDC, custom:Connector_01x01_CastellatedEdge, symbol custom:Connector_01x01_CastellatedEdge
- added J48: +3V3, custom:Connector_01x01_CastellatedEdge, symbol custom:Connector_01x01_CastellatedEdge
- added J49: +3V3A, custom:Connector_01x01_CastellatedEdge, symbol custom:Connector_01x01_CastellatedEdge
- added J50: GND, custom:Connector_01x01_CastellatedEdge, symbol custom:Connector_01x01_CastellatedEdge
- added J51: GNDA, custom:Connector_01x01_CastellatedEdge, symbol custom:Connector_01x01_CastellatedEdge
- added J52: IN_L, custom:Connector_01x01_CastellatedEdge, symbol custom:Connector_01x01_CastellatedEdge
- added J53: IN_R, custom:Connector_01x01_CastellatedEdge, symbol custom:Connector_01x01_CastellatedEdge
- added J54: OUT_L, custom:Connector_01x01_CastellatedEdge, symbol custom:Connector_01x01_CastellatedEdge
- added J55: OUT_R, custom:Connector_01x01_CastellatedEdge, symbol custom:Connector_01x01_CastellatedEdge
- added JP2: SolderJumper_2_Open, Jumper:SolderJumper-2_P1.3mm_Open_RoundedPad1.0x1.5mm, symbol Jumper:SolderJumper_2_Open
- added R7: 10k, symbol Device:R_US
Connections:
- net CODEC_ERROR is gone; now on net SSI_ERROR: TP2.1, U2.11 (GPO)
- net +3V3: now also IC1.C7 (P208/T_DI), J48.1, R7.1
- net +3V3A: now also J49.1
- net GND: now also J45.5 (GND), J50.1, JP2.1 (A)
- net GNDA: now also J51.1
- net IN_L: now also J52.1
- net IN_R: now also J53.1
- net OUT_L: now also J54.1
- net OUT_R: now also J55.1
- net VBUS: now also J45.1 (VCC)
- net SWDIO: now reaches IC1.C6 (P210/TMS/SWDIO)
- net SWDIO: now also J45.2 (SWDIO)
- net ~{RESET}: now reaches IC1.D5 (RES)
- net ~{RESET}: now also J45.3 (~{RESET}), JP2.2 (B), R7.2
- net SWCLK: now reaches IC1.D6 (P211/TCK/SWCLK)
- net SWCLK: now also J45.4 (SWCLK)
- net SWO: now reaches IC1.E7 (P209/TDO)
- net SWO: now also J45.6 (SWO)
- net SSI_ERROR: now reaches IC1.F16 (P707)
- net +9V: no longer names the net of D2.2 (A)
- net +9V: now also J46.1
- net VDC: no longer names the net of C56.1, D1.1 (K), D2.1 (K), U1.6 (VIN), U1.7 (EN)
- net VDC: now also J47.1
- no-connect marks 12 -> 108
Other:
- moved on the sheet: R5, R6

Commit message: choose some parts and start routing
Parts:
- removed L1, L2: 2.2u, symbol Device:L
- added L1, L3: LQH44PN2R2MPRL, vendor:MURATA_LQH44PN2R2MPRL, symbol vendor:LQH44PN2R2MPRL
- C1, C10, C11, C12, C13, C14, C15, C2, C3, C35, C4, C5, C58, C6, C7, C8, C9: footprint (none) -> Capacitor_SMD:C_0402_1005Metric
- C16: renamed from C56; value 4.7u -> 4.7u GRM21BR71E475KA73L; footprint (none) -> Capacitor_SMD:C_0805_2012Metric
- C17: renamed from C45; footprint (none) -> Capacitor_SMD:C_0402_1005Metric
- C18: renamed from C16; value 22u -> 22u GRM21BR61E226ME44L; footprint (none) -> Capacitor_SMD:C_0805_2012Metric
- C19: renamed from C17; footprint (none) -> Capacitor_SMD:C_0402_1005Metric
- C20: renamed from C52; footprint (none) -> Capacitor_SMD:C_0402_1005Metric
- C21: renamed from C57; value 22u -> 22u GRM21BR61E226ME44L; footprint (none) -> Capacitor_SMD:C_0805_2012Metric
- C22: renamed from C18; footprint (none) -> Capacitor_SMD:C_0402_1005Metric
- C23: renamed from C31; footprint (none) -> Capacitor_SMD:C_0402_1005Metric
- C24: renamed from C19; footprint (none) -> Capacitor_SMD:C_0402_1005Metric
- C25: renamed from C32; footprint (none) -> Capacitor_SMD:C_0402_1005Metric
- C26: renamed from C20; footprint (none) -> Capacitor_SMD:C_0402_1005Metric
- C27: renamed from C33; footprint (none) -> Capacitor_SMD:C_0402_1005Metric
- C28: renamed from C21; footprint (none) -> Capacitor_SMD:C_0402_1005Metric
- C29: renamed from C34; footprint (none) -> Capacitor_SMD:C_0402_1005Metric
- C30: renamed from C47; footprint (none) -> Capacitor_SMD:C_0805_2012Metric
- C31: renamed from C53; footprint (none) -> Capacitor_SMD:C_0805_2012Metric
- C32: renamed from C54; footprint (none) -> Capacitor_SMD:C_0805_2012Metric
- C33: renamed from C55; footprint (none) -> Capacitor_SMD:C_0805_2012Metric
- C34: renamed from C22; footprint (none) -> Capacitor_SMD:C_0402_1005Metric
- C36: renamed from C23; footprint (none) -> Capacitor_SMD:C_0402_1005Metric
- C37: renamed from C36; footprint (none) -> Capacitor_SMD:C_0402_1005Metric
- C38: renamed from C46; footprint (none) -> Capacitor_SMD:C_0805_2012Metric
- C39: renamed from C24; footprint (none) -> Capacitor_SMD:C_0402_1005Metric
- C40: renamed from C37; footprint (none) -> Capacitor_SMD:C_0402_1005Metric
- C41: renamed from C48; footprint (none) -> Capacitor_SMD:C_0402_1005Metric
- C42: renamed from C25; footprint (none) -> Capacitor_SMD:C_0402_1005Metric
- C43: renamed from C38; footprint (none) -> Capacitor_SMD:C_0402_1005Metric
- C44: renamed from C26; footprint (none) -> Capacitor_SMD:C_0402_1005Metric
- C45: renamed from C39; footprint (none) -> Capacitor_SMD:C_0402_1005Metric
- C46: renamed from C27; footprint (none) -> Capacitor_SMD:C_0402_1005Metric
- C47: renamed from C40; footprint (none) -> Capacitor_SMD:C_0402_1005Metric
- C48: renamed from C28; footprint (none) -> Capacitor_SMD:C_0402_1005Metric
- C49: renamed from C41; footprint (none) -> Capacitor_SMD:C_0402_1005Metric
- C50: renamed from C51; footprint (none) -> Capacitor_SMD:C_0402_1005Metric
- C51: renamed from C50; footprint (none) -> Capacitor_SMD:C_0402_1005Metric
- C52: renamed from C49; footprint (none) -> Capacitor_SMD:C_0805_2012Metric
- C53: renamed from C29; footprint (none) -> Capacitor_SMD:C_0402_1005Metric
- C54: renamed from C42; footprint (none) -> Capacitor_SMD:C_0402_1005Metric
- C55: renamed from C59; footprint (none) -> Capacitor_SMD:C_0402_1005Metric
- C56: renamed from C43; footprint (none) -> Capacitor_SMD:C_0402_1005Metric
- C57: renamed from C44; footprint (none) -> Capacitor_SMD:C_0402_1005Metric
- C59: renamed from C30; value 47u -> 47u GRM31CR61E476ME44L; footprint (none) -> Capacitor_SMD:C_1206_3216Metric
- D1: renamed from D2; value D -> RB161M-20TR; footprint (none) -> Diode_SMD:D_SOD-123
- D2: renamed from D1; value D -> RB161M-20TR; footprint (none) -> Diode_SMD:D_SOD-123
- JP2: renamed from JP1; footprint (none) -> Jumper:SolderJumper-2_P1.3mm_Bridged_RoundedPad1.0x1.5mm
- R1: renamed from R5; footprint (none) -> Resistor_SMD:R_0402_1005Metric
- R2: renamed from R6; footprint (none) -> Resistor_SMD:R_0402_1005Metric
- R3: renamed from R4; footprint (none) -> Resistor_SMD:R_0402_1005Metric
- R4: renamed from R7; footprint (none) -> Resistor_SMD:R_0402_1005Metric
- R5: renamed from R1; footprint (none) -> Resistor_SMD:R_0402_1005Metric
- R6: renamed from R2; footprint (none) -> Resistor_SMD:R_0402_1005Metric
- R7: renamed from R3; footprint (none) -> Resistor_SMD:R_0402_1005Metric
- TP1: renamed from TP2; footprint (none) -> TestPoint:TestPoint_Pad_1.0x1.0mm
- TP2: renamed from TP1; footprint (none) -> TestPoint:TestPoint_Pad_1.0x1.0mm
- renumbered J30 to J1, J25 to J10, J38 to J11, J37 to J12, J1 to J13, J8 to J14, J26 to J15, J42 to J16, J43 to J17, J28 to J18, J29 to J19, J21 to J2, J31 to J20, J10 to J21, J12 to J22, J41 to J23, J34 to J24, J33 to J25, J13 to J26, J9 to J27, J36 to J28, J39 to J29, J20 to J3, J14 to J30, J16 to J31, J2 to J32, J35 to J33, J32 to J34, J44 to J35, J17 to J36, J15 to J37, J27 to J38, J4 to J39, J24 to J4, J3 to J40, J5 to J41, J6 to J42, J7 to J43, J11 to J44, J46 to J45, J47 to J46, J45 to J47, J40 to J5, J19 to J6, J23 to J7, J22 to J8, J18 to J9, JP2 to JP1
Connections:
- net +0V9: now also L1.2
- net +3V3: now also L3.2
- net VLO: now also L1.1
- net at U1.4 (SW): now also L3.1
Other:
- note removed: "max inductor current should be ~1.16 A, so saturate at 20% above that and choose output cap. see tables 9-4 & 9-5 in the datasheet for recommended parts; output cap is not specified, but they recommend X7R/X5R, low ESR/ESL"
- moved on the sheet: C18, C19, C21
