File: hardware/projects/octaver/octaver.kicad_sch (KiCad schematic)
At the start: 53 parts, among them J1 In, J2 Out, J3 Power, J4 pot_hp, J5 sw_hp, J6 fs_hp, J7 sw_hp2, SW1 Integrator On, SW2 stable / alive, SW3 Differentiator On, SW4 Octave Lo/Hi, SW6 Footswitch, U1 TL072, U2 TL072, U3 TL072, U5 LM311, U6 40175, U7 AD633JNZ

Commit message: update octaver/ with new library names
Parts:
- J1, J2: footprint circuits:mono_jack -> custom:mono_jack
- RV2, RV3, RV5, RV6, RV7, RV8: footprint circuits:Taiss_Potentiometer_vertical -> custom:Taiss_Potentiometer_vertical
- SW1, SW2, SW3, SW4: footprint circuits:Adam Tech SW-T3-2B-A-A3-S1 -> custom:Adam Tech SW-T3-2B-A-A3-S1
- SW6: footprint circuits:PBS-24-302_3PDT -> custom:PBS-24-302_3PDT
- U7: footprint footprints:N_8_ADI -> Package_DIP:DIP-8_W7.62mm
Changed lines of the file:
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@@
 			)
 		)
-		(property "Footprint" "circuits:mono_jack"
+		(property "Footprint" "custom:mono_jack"
 			(at 105.41 73.66 0)
 			(hide yes)
@@
 			)
 		)
-		(property "Footprint" "footprints:N_8_ADI"
+		(property "Footprint" "Package_DIP:DIP-8_W7.62mm"
 			(at 260.35 157.48 0)
 			(hide yes)
@@
 			)
 		)
-		(property "Footprint" "circuits:Taiss_Potentiometer_vertical"
+		(property "Footprint" "custom:Taiss_Potentiometer_vertical"
 			(at 242.57 87.63 0)
 			(hide yes)
@@
 			)
 		)
-		(property "Footprint" "circuits:mono_jack"
+		(property "Footprint" "custom:mono_jack"
 			(at 105.41 59.69 0)
 			(hide yes)
@@
 			)
 		)
-		(property "Footprint" "circuits:Taiss_Potentiometer_vertical"
+		(property "Footprint" "custom:Taiss_Potentiometer_vertical"
 			(at 302.26 59.69 0)
 			(hide yes)
@@
 			)
 		)
-		(property "Footprint" "circuits:Taiss_Potentiometer_vertical"
+		(property "Footprint" "custom:Taiss_Potentiometer_vertical"
 			(at 154.94 142.24 0)
 			(hide yes)
@@
 			)
 		)
-		(property "Footprint" "circuits:Adam Tech SW-T3-2B-A-A3-S1"
+		(property "Footprint" "custom:Adam Tech SW-T3-2B-A-A3-S1"
 			(at 137.16 92.71 0)
 			(hide yes)
@@
 			)
 		)
-		(property "Footprint" "circuits:Adam Tech SW-T3-2B-A-A3-S1"
+		(property "Footprint" "custom:Adam Tech SW-T3-2B-A-A3-S1"
 			(at 158.75 165.1 0)
 			(hide yes)
@@
 			)
 		)
-		(property "Footprint" "circuits:Taiss_Potentiometer_vertical"
+		(property "Footprint" "custom:Taiss_Potentiometer_vertical"
 			(at 290.83 93.98 0)
 			(hide yes)
@@
 			)
 		)
-		(property "Footprint" "circuits:PBS-24-302_3PDT"
+		(property "Footprint" "custom:PBS-24-302_3PDT"
 			(at 43.18 68.58 0)
 			(hide yes)
@@
 			)
 		)
-		(property "Footprint" "circuits:PBS-24-302_3PDT"
+		(property "Footprint" "custom:PBS-24-302_3PDT"
 			(at 43.18 83.82 0)
 			(hide yes)
@@
 			)
 		)
-		(property "Footprint" "circuits:PBS-24-302_3PDT"
+		(property "Footprint" "custom:PBS-24-302_3PDT"
 			(at 44.45 203.2 0)
 			(hide yes)
@@
 			)
 		)
-		(property "Footprint" "circuits:Adam Tech SW-T3-2B-A-A3-S1"
+		(property "Footprint" "custom:Adam Tech SW-T3-2B-A-A3-S1"
 			(at 237.49 180.34 0)
 			(hide yes)
@@
 			)
 		)
-		(property "Footprint" "circuits:Taiss_Potentiometer_vertical"
+		(property "Footprint" "custom:Taiss_Potentiometer_vertical"
 			(at 241.3 157.48 0)
 			(hide yes)
@@
 			)
 		)
-		(property "Footprint" "circuits:Taiss_Potentiometer_vertical"
+		(property "Footprint" "custom:Taiss_Potentiometer_vertical"
 			(at 356.87 97.79 0)
 			(hide yes)
@@
 			)
 		)
-		(property "Footprint" "circuits:Adam Tech SW-T3-2B-A-A3-S1"
+		(property "Footprint" "custom:Adam Tech SW-T3-2B-A-A3-S1"
 			(at 227.33 71.12 0)
 			(hide yes)

Commit message: make some edits & add some comments
Parts:
- added B1, B2, B3: MouseBite, Panelization:MouseBite-Slot_2.54x2.54mm_on-edge_D0.5mm_P0.85mm_4h_Trace, symbol Mechanical:MouseBite
Changed lines of the file:
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@@
 	)
 	(symbol
+		(lib_id "Mechanical:MouseBite")
+		(at 185.42 219.71 0)
+		(unit 1)
+		(body_style 1)
+		(exclude_from_sim yes)
+		(in_bom no)
+		(on_board yes)
+		(in_pos_files yes)
+		(dnp no)
+		(fields_autoplaced yes)
+		(property "Reference" "B2"
+			(at 187.96 218.5024 0)
+			(show_name no)
+			(do_not_autoplace no)
+			(effects
+				(font
+					(size 1.27 1.27)
+				)
+				(justify left)
+			)
+		)
+		(property "Value" "MouseBite"
+			(at 187.96 221.0424 0)
+			(show_name no)
+			(do_not_autoplace no)
+			(effects
+				(font
+					(size 1.27 1.27)
+				)
+				(justify left)
+			)
+		)
+		(property "Footprint" "Panelization:MouseBite-Slot_2.54x2.54mm_on-edge_D0.5mm_P0.85mm_4h_Trace"
+			(at 185.42 219.71 0)
+			(hide yes)
+			(show_name no)
+			(do_not_autoplace no)
+			(effects
+				(font
+					(size 1.27 1.27)
+				)
+			)
+		)
+		(property "Datasheet" ""
+			(at 185.42 219.71 0)
+			(hide yes)
+			(show_name no)
+			(do_not_autoplace no)
+			(effects
+				(font
+					(size 1.27 1.27)
+				)
+			)
+		)
+		(property "Description" "Mouse bites, break lines"
+			(at 185.42 219.71 0)
+			(hide yes)
+			(show_name no)
+			(do_not_autoplace no)
+			(effects
+				(font
+					(size 1.27 1.27)
+				)
+			)
+		)
+		(instances
+			(project "octaver"
+				(path "/14f76e9a-222a-4860-b13d-facccb28af95"
+					(reference "B2")
+					(unit 1)
+				)
+			)
+		)
+	)
+	(symbol
 		(lib_id "power:GND")
 		(at 137.16 137.16 0)
@@
 	)
 	(symbol
+		(lib_id "Mechanical:MouseBite")
+		(at 185.42 231.14 0)
+		(unit 1)
+		(body_style 1)
+		(exclude_from_sim yes)
+		(in_bom no)
+		(on_board yes)
+		(in_pos_files yes)
+		(dnp no)
+		(fields_autoplaced yes)
+		(property "Reference" "B3"
+			(at 187.96 229.9324 0)
+			(show_name no)
+			(do_not_autoplace no)
+			(effects
+				(font
+					(size 1.27 1.27)
+				)
+				(justify left)
+			)
+		)
+		(property "Value" "MouseBite"
+			(at 187.96 232.4724 0)
+			(show_name no)
+			(do_not_autoplace no)
+			(effects
+				(font
+					(size 1.27 1.27)
+				)
+				(justify left)
+			)
+		)
+		(property "Footprint" "Panelization:MouseBite-Slot_2.54x2.54mm_on-edge_D0.5mm_P0.85mm_4h_Trace"
+			(at 185.42 231.14 0)
+			(hide yes)
+			(show_name no)
+			(do_not_autoplace no)
+			(effects
+				(font
+					(size 1.27 1.27)
+				)
+			)
+		)
+		(property "Datasheet" ""
+			(at 185.42 231.14 0)
+			(hide yes)
+			(show_name no)
+			(do_not_autoplace no)
+			(effects
+				(font
+					(size 1.27 1.27)
+				)
+			)
+		)
+		(property "Description" "Mouse bites, break lines"
+			(at 185.42 231.14 0)
+			(hide yes)
+			(show_name no)
+			(do_not_autoplace no)
+			(effects
+				(font
+					(size 1.27 1.27)
+				)
+			)
+		)
+		(instances
+			(project "octaver"
+				(path "/14f76e9a-222a-4860-b13d-facccb28af95"
+					(reference "B3")
+					(unit 1)
+				)
+			)
+		)
+	)
+	(symbol
 		(lib_id "symbols:Conn_01x10_10part")
 		(at 346.71 88.9 90)
@@
 				)
 			)
+		)
+	)
+	(symbol
+		(lib_id "Mechanical:MouseBite")
+		(at 185.42 208.28 0)
+		(unit 1)
+		(body_style 1)
+		(exclude_from_sim yes)
+		(in_bom no)
+		(on_board yes)
+		(in_pos_files yes)
+		(dnp no)
+		(fields_autoplaced yes)
+		(property "Reference" "B1"
+			(at 187.96 207.0724 0)
+			(show_name no)
+			(do_not_autoplace no)
+			(effects
+				(font
+					(size 1.27 1.27)
+				)
+				(justify left)
+			)
+		)
+		(property "Value" "MouseBite"
+			(at 187.96 209.6124 0)
+			(show_name no)
+			(do_not_autoplace no)
+			(effects
+				(font
+					(size 1.27 1.27)
+				)
+				(justify left)
+			)
+		)
+		(property "Footprint" "Panelization:MouseBite-Slot_2.54x2.54mm_on-edge_D0.5mm_P0.85mm_4h_Trace"
+			(at 185.42 208.28 0)
+			(hide yes)
+			(show_name no)
+			(do_not_autoplace no)
+			(effects
+				(font
+					(size 1.27 1.27)
+				)
+			)
+		)
+		(property "Datasheet" ""
+			(at 185.42 208.28 0)
+			(hide yes)
+			(show_name no)
+			(do_not_autoplace no)
+			(effects
+				(font
+					(size 1.27 1.27)
+				)
+			)
+		)
+		(property "Description" "Mouse bites, break lines"
+			(at 185.42 208.28 0)
+			(hide yes)
+			(show_name no)
+			(do_not_autoplace no)
+			(effects
+				(font
+					(size 1.27 1.27)
+				)
+			)
+		)
+		(instances
+			(project "octaver"
+				(path "/14f76e9a-222a-4860-b13d-facccb28af95"
+					(reference "B1")
+					(unit 1)
+				)
+			)

Commit message: make final (?) major edits
Parts:
- B1, B2, B3: footprint Panelization:MouseBite-Slot_2.54x2.54mm_on-edge_D0.5mm_P0.85mm_4h_Trace -> custom:MouseBite_2.54x7.62mm_JLCPCB
Changed lines of the file:
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@@
 			)
 		)
-		(property "Footprint" "Panelization:MouseBite-Slot_2.54x2.54mm_on-edge_D0.5mm_P0.85mm_4h_Trace"
+		(property "Footprint" "custom:MouseBite_2.54x7.62mm_JLCPCB"
 			(at 185.42 219.71 0)
 			(hide yes)
@@
 			)
 		)
-		(property "Footprint" "Panelization:MouseBite-Slot_2.54x2.54mm_on-edge_D0.5mm_P0.85mm_4h_Trace"
+		(property "Footprint" "custom:MouseBite_2.54x7.62mm_JLCPCB"
 			(at 185.42 231.14 0)
 			(hide yes)
@@
 			)
 		)
-		(property "Footprint" "Panelization:MouseBite-Slot_2.54x2.54mm_on-edge_D0.5mm_P0.85mm_4h_Trace"
+		(property "Footprint" "custom:MouseBite_2.54x7.62mm_JLCPCB"
 			(at 185.42 208.28 0)
 			(hide yes)

Commit message: octaver: Most of the rev2 fixes
Most notably, fixed the whine by switching pre-gain to an inverting amp
Parts:
- removed J6: fs_hp, Connector_PinHeader_2.54mm:PinHeader_1x05_P2.54mm_Vertical, symbol symbols:Conn_01x5_5part
- removed J7: sw_hp2, Connector_PinHeader_2.54mm:PinHeader_1x05_P2.54mm_Vertical, symbol symbols:Conn_01x5_5part
- added C11: 10p, Capacitor_SMD:C_0603_1608Metric, symbol Device:C_Small
- added J8: main board, Connector_PinHeader_2.54mm:PinHeader_1x04_P2.54mm_Vertical, symbol Connector_Generic:Conn_01x04
- added J9: fs board, Connector_PinHeader_2.54mm:PinHeader_1x04_P2.54mm_Vertical, symbol Connector_Generic:Conn_01x04
- RV5: value A100K -> C100K
- RV8: value A1M -> C1M
Connections:
- net fsgnd is gone; now on net fs_gndpwr: J1.S, J2.S
- net +9V: now also J8.2 (Pin_2)
- net GND: now also U2.3 (+); no longer R5.2
- net GNDPWR: now also J8.3 (Pin_3)
- net circuit_in: now also J8.1 (Pin_1)
- net circuit_out: now also J8.4 (Pin_4)
- net pot_gnd: now also RV2.1; no longer RV2.3
- net at C9.2, J5.7 (Pin_3), U3.1: now also C11.2
- net at J5.6 (Pin_3), R19.1, U3.2 (-): now also C11.1
- net fs_pwr: now reaches SW6.8 (B)
- net fs_pwr: now also J9.2 (Pin_2)
- net live: now reaches R11.2, R9.2, SW2.3 (C), U5.2 (+)
- net octave_hi: now reaches R11.1, R12.1, SW4.3 (C), U5.7, U6.9 (Ck)
- net diff bypass: now reaches C5.2, R10.2, U7.7 (W)
- net diff bypass: now also SW3.1 (A); no longer SW3.3 (C)
- net at SW1.2 (B): now also R5.2; no longer U2.3 (+)
- net at J4.9 (Pin_3): now also RV2.3; no longer RV2.1
- net at J4.4 (Pin_3): now also RV3.1; no longer RV3.3
- net diff on: now reaches C6.1, R13.1, U1.7
- net diff on: now also SW3.3 (C); no longer SW3.1 (A)
- net at RV5.1: no longer R15.2
- net at RV5.3: now also R15.2
- net int_on: now reaches C2.1, R4.1, U2.7
- net int_on: now also SW1.3 (C); no longer SW1.1 (A)
- net at C8.2, RV8.3: now also RV3.3; no longer RV3.1
- net int_off: now reaches J5.4 (Pin_3), R3.2, U1.1, U1.2 (-)
- net int_off: now also SW1.1 (A); no longer SW1.3 (C)
- net stable: now reaches SW2.1 (A)
- net octave_lo: now reaches SW4.1 (A), U6.13, U6.14
- net fs_gndpwr: now reaches D1.1 (K)
- net fs_gndpwr: now also J9.3 (Pin_3)
- net fs_in: now reaches SW6.3 (C)
- net fs_in: now also J9.1 (Pin_1)
- net fs_out: now reaches SW6.6 (C)
- net fs_out: now also J9.4 (Pin_4)
Other:
- moved on the sheet: R5, RV5, SW1, SW3
